File: due/osciloador/kicad/oscila_mag.kicad_pcb (KiCad board)
At the start: 2 copper layers, 36 parts, among them P3 Analog, P5 PWM, P6 PWM, Q1 BC548, U1 TC4420CPA, U2 TC4420CPA

Commit message: Update due/osciloador/kicad/
Signed-off-by: Felipe Leon <fglfgl27@gmail.com>
Parts:
- removed R6, R7: 100k, Resistor_THT:R_Axial_DIN0207_L6.3mm_D2.5mm_P10.16mm_Horizontal
- removed REF**: BarrelJack_Horizontal, Connector_BarrelJack:BarrelJack_Horizontal
- added C5: 1u, Capacitor_THT:C_Disc_D8.0mm_W5.0mm_P10.00mm, F.Cu at (114.3, 47.8)
- added C6: 1u, Capacitor_THT:C_Disc_D8.0mm_W5.0mm_P10.00mm, F.Cu at (113.3, 124.0)
- C1, C4: value 1000u -> 222n
- L1, L2: value INDUCTOR -> 50u
- R1, R3: value 47R -> 150
- R5, R9: value 10k -> 4.7k
Connections:
- net ADC_L1 renamed ADC_0_L1
- net ADC_L2 renamed ADC_7_L2
- net PWM6 renamed PWM4
Routing:
- net PWM6: track 0.00 -> 9.21 mm
- net PWM4: track 9.21 -> 0.00 mm
