File: uno/am/am/ci_KiCad/ci.sch (KiCad schematic (older format))
At the start: 9 parts

Commit message: Update AM project
Signed-off-by: fgl27 <fglfgl27@gmail.com>
Parts:
- added C3: 447 pF, symbol pspice:CAP
- added GND: GNDREF, symbol power:GNDREF
- added POT1: 1k Ω, symbol Device:R_POT
- C1: value CAP 10 μ -> 10 μF
- R1, R2: value R 10k Ω -> 10k Ω
Connections:
- net GNDREF: now also C3.2, GND.1 (GNDREF)
- net at A1.26 (D11): now also POT1.3; no longer A1.1 (A)
- new net: A1.1 (A), C3.1, POT1.1, POT1.2
Other:
- note added: "Saída antena e um filtro passa baixa ajustavel\nFrequência de corte 800kHz R = 445,06 Ω"
- moved on the sheet: A1
Changed lines of the file:
@@
 L Device:Antenna A1
 U 1 1 605397BD
-P 4900 4050
-F 0 "A1" H 4980 4039 50  0000 L CNN
-F 1 "Antena" H 4980 3948 50  0000 L CNN
-F 2 "" H 4900 4050 50  0001 C CNN
-F 3 "~" H 4900 4050 50  0001 C CNN
-	1    4900 4050
+P 4500 3900
+F 0 "A1" H 4450 4250 50  0000 L CNN
+F 1 "Antena" H 4400 4100 50  0000 L CNN
+F 2 "" H 4500 3900 50  0001 C CNN
+F 3 "~" H 4500 3900 50  0001 C CNN
+	1    4500 3900
 	1    0    0    -1
 $EndComp
@@
 P 6950 3550
 F 0 "R1" H 7020 3596 50  0000 L CNN
-F 1 "R 10k Ω" H 7020 3505 50  0000 L CNN
+F 1 "10k Ω" H 7020 3505 50  0000 L CNN
 F 2 "" V 6880 3550 50  0001 C CNN
 F 3 "~" H 6950 3550 50  0001 C CNN
@@
 P 7650 3800
 F 0 "C1" V 7965 3800 50  0000 C CNN
-F 1 "CAP 10 μ" V 7874 3800 50  0000 C CNN
+F 1 "10 μF" V 7874 3800 50  0000 C CNN
 F 2 "" H 7650 3800 50  0001 C CNN
 F 3 "~" H 7650 3800 50  0001 C CNN
@@
 P 6950 4000
 F 0 "R2" H 7020 4046 50  0000 L CNN
-F 1 "R 10k Ω" H 7020 3955 50  0000 L CNN
+F 1 "10k Ω" H 7020 3955 50  0000 L CNN
 F 2 "" V 6880 4000 50  0001 C CNN
 F 3 "~" H 6950 4000 50  0001 C CNN
@@
 Wire Wire Line
 	5850 2800 5850 2600
-Wire Wire Line
-	5450 4300 4900 4300
-Wire Wire Line
-	4900 4300 4900 4250
 Wire Wire Line
 	6950 3700 6950 3800
@@
 Wire Wire Line
 	6050 5100 6050 4900
+$Comp
+L pspice:CAP C3
+U 1 1 60911131
+P 4500 4650
+F 0 "C3" H 4815 4650 50  0000 C CNN
+F 1 "447 pF" H 4850 4550 50  0000 C CNN
+F 2 "" H 4500 4650 50  0001 C CNN
+F 3 "~" H 4500 4650 50  0001 C CNN
+	1    4500 4650
+	1    0    0    -1
+$EndComp
+$Comp
+L power:GNDREF GND
+U 1 1 609123E8
+P 4500 5150
+F 0 "GND" H 4450 4950 50  0000 L CNN
+F 1 "GNDREF" H 4505 4977 50  0001 C CNN
+F 2 "" H 4500 5150 50  0001 C CNN
+F 3 "" H 4500 5150 50  0001 C CNN
+	1    4500 5150
+	1    0    0    -1
+$EndComp
+Wire Wire Line
+	4500 4900 4500 5150
+$Comp
+L Device:R_POT POT1
+U 1 1 60921746
+P 5050 4300
+F 0 "POT1" V 4935 4300 50  0000 C CNN
+F 1 "1k Ω" V 4844 4300 50  0000 C CNN
+F 2 "" H 5050 4300 50  0001 C CNN
+F 3 "~" H 5050 4300 50  0001 C CNN
+	1    5050 4300
+	0    -1   -1   0
+$EndComp
+Wire Wire Line
+	5200 4300 5450 4300
+Wire Wire Line
+	4900 4300 4850 4300
+Wire Wire Line
+	4500 4100 4500 4300
+Connection ~ 4500 4300
+Wire Wire Line
+	5050 4150 4850 4150
+Wire Wire Line
+	4850 4150 4850 4300
+Connection ~ 4850 4300
+Wire Wire Line
+	4850 4300 4500 4300
+Wire Wire Line
+	4500 4300 4500 4400
+Text Notes 3400 3400 0    50   ~ 0
+Saída antena e um filtro passa baixa ajustavel\nFrequência de corte 800kHz R = 445,06 Ω
 $EndSCHEMATC
